File: RPUlux/17323^1.brd (EAGLE design)
At the start: 73.7 x 73.7 mm, 137 parts, among them J1 PST1,0/6-3,5, J10 ICSP, J11 S04B, J12 FRIEND, J2 PST1,0/6-3,5, J3 PST1,0/6-3,5, J4 PPPC101LFBN, J5 PPPC081LFBN, J6 PST1,0/2-3,5, J7 PST1,0/3-3,5, J8 PPPC101LFBN, J9 PPPC101LFBN, Q1 K1N, Q10 K1N, Q11 K38, Q12 K3N, Q13 K3N, Q14 34N, Q15 34N, Q16 K1N, Q17 K38, Q18 K3N, Q19 K38, Q2 P65, Q20 K1N, Q22 K38, Q23 K38, Q24 K3N, Q3 K38, Q4 P65, Q5 K3N, Q6 K1N, Q7 K3N, Q8 P65, Q9 K38, U1 1087, U2 I50115, U3 A6, U4 A6, U5 A6, U6 A6, U7 A6, U8 A6, U9 ATMEGA328PB-AU, Y1 16MHz

Commit message: RPUlux: ^1 schmatic update
Parts:
- R18, R20, R22, R29, R31, R33: value 0.3 -> 0.15
Changed lines of the file:
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@@
 <attribute name="VALUE" x="43.053" y="20.701" size="0.4064" layer="27" rot="R270"/>
 </element>
-<element name="R18" library="R-C" package="C1210(3225)" value="0.3" x="46.863" y="12.065" smashed="yes">
+<element name="R18" library="R-C" package="C1210(3225)" value="0.15" x="46.863" y="12.065" smashed="yes">
 <attribute name="NAME" x="45.466" y="9.779" size="0.6096" layer="25"/>
 <attribute name="VALUE" x="45.847" y="11.811" size="0.4064" layer="27"/>
@@
 <attribute name="VALUE" x="18.3560125" y="21.001221875" size="0.4064" layer="27" rot="R225"/>
 </element>
-<element name="R29" library="R-C" package="C1210(3225)" value="0.3" x="21.717" y="12.573" smashed="yes">
+<element name="R29" library="R-C" package="C1210(3225)" value="0.15" x="21.717" y="12.573" smashed="yes">
 <attribute name="NAME" x="22.86" y="10.795" size="0.6096" layer="25" rot="R180"/>
 <attribute name="VALUE" x="21.082" y="12.192" size="0.4064" layer="27"/>
@@
 <attribute name="VALUE" x="35.433" y="11.176" size="0.4064" layer="27" rot="R180"/>
 </element>
-<element name="R20" library="R-C" package="C1210(3225)" value="0.3" x="38.608" y="12.7" smashed="yes">
+<element name="R20" library="R-C" package="C1210(3225)" value="0.15" x="38.608" y="12.7" smashed="yes">
 <attribute name="NAME" x="39.37" y="10.922" size="0.6096" layer="25" rot="R180"/>
 <attribute name="VALUE" x="37.592" y="12.446" size="0.4064" layer="27"/>
@@
 <attribute name="VALUE" x="9.271" y="12.573" size="0.4064" layer="27" rot="R270"/>
 </element>
-<element name="R31" library="R-C" package="C1210(3225)" value="0.3" x="14.351" y="12.192" smashed="yes">
+<element name="R31" library="R-C" package="C1210(3225)" value="0.15" x="14.351" y="12.192" smashed="yes">
 <attribute name="NAME" x="13.462" y="10.033" size="0.6096" layer="25"/>
 <attribute name="VALUE" x="13.335" y="11.938" size="0.4064" layer="27"/>
@@
 <attribute name="VALUE" x="27.051" y="11.43" size="0.4064" layer="27" rot="R180"/>
 </element>
-<element name="R22" library="R-C" package="C1210(3225)" value="0.3" x="30.353" y="12.573" smashed="yes">
+<element name="R22" library="R-C" package="C1210(3225)" value="0.15" x="30.353" y="12.573" smashed="yes">
 <attribute name="NAME" x="31.115" y="10.922" size="0.6096" layer="25" rot="R180"/>
 <attribute name="VALUE" x="29.337" y="12.319" size="0.4064" layer="27"/>
@@
 <attribute name="VALUE" x="4.445" y="11.049" size="0.4064" layer="27" rot="R180"/>
 </element>
-<element name="R33" library="R-C" package="C1210(3225)" value="0.3" x="5.588" y="13.589" smashed="yes">
+<element name="R33" library="R-C" package="C1210(3225)" value="0.15" x="5.588" y="13.589" smashed="yes">
 <attribute name="NAME" x="7.239" y="11.43" size="0.6096" layer="25" rot="R180"/>
 <attribute name="VALUE" x="4.572" y="13.335" size="0.4064" layer="27"/>
