File: Gravimetric/17341.brd (EAGLE design)
At the start: 110.5 x 72.4 mm, 279 parts, among them J1 PST1,0/2-3,5, J10 RJ45J, J12 ICSP, J13 S04B, J14 FRIEND, J2 PST1,0/6-3,5, J3 PST1,0/3-3,5, J5 PST1,0/5-3,5, J6 PST1,0/5-3,5, J7 Pi Zero, J8 PST1,0/3-3,5, J9 RJ45J, Q1 IRFR5305, Q10 K38, Q101 K3N, Q102 K3N, Q103 K3N, Q104 K3N, Q105 K38, Q106 K1N, Q107 K3N, Q108 K3N, Q109 K1N, Q11 K38, Q110 K1N, Q111 K1N, Q112 K1N, Q113 K1N, Q114 K1N, Q115 K1N, Q116 K3N, Q117 K3N, Q118 K38, Q119 K3N, Q120 K3N, Q121 K1N, Q122 K38, Q123 K3N, Q124 K3N, Q125 K1N, Q126 K38, Q127 K3N, Q128 K3N, Q129 K1N, Q130 K1N, Q131 K1N, Q132 K38, Q133 K3N, Q134 K3N, Q135 K1N, Q136 K1N, Q137 K38, Q138 K3N, Q139 K3N, Q140 K1N, Q141 K1N, Q142 K1N, Q143 K38, Q144 K38, Q145 K3N, Q146 K1N, Q147 K3N, Q148 K1N, Q149 K1N, Q150 K1N, Q151 K1N, Q152 K38, Q153 K38, Q2 K1N, Q201 K1N, Q202 K1N, Q203 K1N, Q3 IRFR5305, Q4 P65, Q5 K3N, Q6 K1N, Q7 K3N, Q8 P65, Q9 K38, U1 1087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

Commit message: Gravimetric: ^2 wip
Parts:
- added TP1, TP2: TPPAD1-08, J-TP:P1-08
- moved R237 8.33 mm to (58.1, 27.4), turned to 180 degrees
- moved R235 1.76 mm to (80.3, 52.3), turned to 180 degrees
- moved R230 0.92 mm to (74.0, 48.4)
Connections:
- net CS_DIVERSION: now also Q118.3(D); no longer Q118.2(S)
- net CS_ICP3: now also Q105.3(D); no longer Q105.2(S)
- net N$42: now also Q105.2(S); no longer Q105.3(D)
- net N$55: now also Q118.2(S); no longer Q118.3(D)
- net N$93: no longer U202.13
- net SCL0: now also TP2.TP
- net SDA0: now also TP1.TP
- net SHUTDWN: now also U202.13
Routing:
- net SHUTDWN: track 3.78 -> 59.8 mm, vias 0 -> 2
- net N$93: track 107.8 -> 57.9 mm, vias 7 -> 4
- net !RESET!: track 70.9 -> 67.6 mm
- net RX0: track 33.8 -> 36.6 mm
- net ICP4: track 100.0 -> 97.2 mm
- net N$78: track 45.9 -> 43.3 mm
- net N$55: track 2.09 -> 4.40 mm
- net MGR_!SS!: track 58.7 -> 60.7 mm
- net TX_DE: track 59.7 -> 61.6 mm
- net DTR_!RE: track 48.4 -> 50.3 mm
- net CS_DIVERSION: track 49.1 -> 50.9 mm
- net CS_ICP3: track 64.6 -> 63.0 mm
- net 0V: track 2.79 -> 4.19 mm, vias 168 -> 171
- net SCL0: track 10.1 -> 11.3 mm
- net N$42: track 14.0 -> 15.2 mm
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Other:
- board text added: "17341^2"
- board text removed: "17341^1"

Commit message: Gravimetric: ^2 oshpark accepted file, now reviewing
Parts:
- moved TP2 0.85 mm to (74.9, 46.6)
Routing:
- net !RESET!: track 67.6 -> 67.1 mm
Other:
- board text added: "REMOVE ALTERNAT POWER BEFOR ISP PROGRAMING"
