File: Gravimetric/17341.sch (EAGLE design)
At the start: 279 parts, among them J1 PST1,0/2-3,5, J10 RJ45J, J12 ICSP, J13 S04B, J14 FRIEND, J2 PST1,0/6-3,5, J3 PST1,0/3-3,5, J5 PST1,0/5-3,5, J6 PST1,0/5-3,5, J7 Pi Zero, J8 PST1,0/3-3,5, J9 RJ45J, Q1 IRFR5305, Q10 K38, Q101 K3N, Q102 K3N, Q103 K3N, Q104 K3N, Q105 K38, Q106 K1N, Q107 K3N, Q108 K3N, Q109 K1N, Q11 K38, Q110 K1N, Q111 K1N, Q112 K1N, Q113 K1N, Q114 K1N, Q115 K1N, Q116 K3N, Q117 K3N, Q118 K38, Q119 K3N, Q120 K3N, Q121 K1N, Q122 K38, Q123 K3N, Q124 K3N, Q125 K1N, Q126 K38, Q127 K3N, Q128 K3N, Q129 K1N, Q130 K1N, Q131 K1N, Q132 K38, Q133 K3N, Q134 K3N, Q135 K1N, Q136 K1N, Q137 K38, Q138 K3N, Q139 K3N, Q140 K1N, Q141 K1N, Q142 K1N, Q143 K38, Q144 K38, Q145 K3N, Q146 K1N, Q147 K3N, Q148 K1N, Q149 K1N, Q150 K1N, Q151 K1N, Q152 K38, Q153 K38, Q2 K1N, Q201 K1N, Q202 K1N, Q203 K1N, Q3 IRFR5305, Q4 P65, Q5 K3N, Q6 K1N, Q7 K3N, Q8 P65, Q9 K38, U1 1087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

Commit message: Gravimetric: ^2 wip
Parts:
- added TP1, TP2: TPPAD1-08, J-TP:TPPAD1-08
Connections:
- net CS_DIVERSION: now also Q118.D; no longer Q118.S
- net CS_ICP3: now also Q105.D; no longer Q105.S
- net N$42: now also Q105.S; no longer Q105.D
- net N$55: now also Q118.S; no longer Q118.D
- net N$93: no longer U202F.I
- net SCL0: now also TP2.TP
- net SDA0: now also TP1.TP
- net SHUTDWN: now also U202F.I
Other:
- note added: "7/16/20"
- note added: "DIVERSON & START CUTOFF SHUTDOWN SW OVERIDE"
- note added: "REMOVE ALTERNAT POWER BEFOR ISP PROGRAMING"
- note added: "^2"
- moved on the sheet: R237

Commit message: Gravimetric: ^2 oshpark accepted file, now reviewing
Other:
- note added: "APPLICATION CONTROLLER"
- note removed: "PROGRAMMABLE CONTROLLER"
Changed lines of the file:
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@@
 <text x="13.97" y="243.078" size="1.778" layer="98">POWER 7-36V</text>
 <text x="133.35" y="245.618" size="1.778" layer="98">BLOCKS -40V</text>
-<text x="117.348" y="153.162" size="2.54" layer="98">PROGRAMMABLE CONTROLLER</text>
+<text x="130.048" y="155.702" size="2.54" layer="98">APPLICATION CONTROLLER</text>
 <text x="60.96" y="110.49" size="1.778" layer="98">ECS-160-20-3X-TR
 16MHZ +/- 30PPM
