File: PiUpdi/19260.sch (EAGLE design)
At the start: 31 parts, among them J1 PPPC101LFBN, J3 PPPC101LFBN, J4 PPPC101LFBN, J5 40 PIN HDR, Q1 DMB, Q2 K38, Q3 K38, Q4 K84, U1 I50115H, U2 Z4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

Commit message: PiUpdi: ^1 layout wip
serial crossover error fixed
Parts:
- added J2: PPPC101LFBN, J-HDR2.54mm:F1X10
- J4: value PPPC101LFBN -> PST1,0/2-3,5; device J-HDR2.54mm:F1X10 -> J-HDR3.5mm:MCV2
Connections:
- removed net N$3: Q3.D, R3.2, R4.2, S1.2
- removed net VIN: C1.1, U1.VIN
- new net N$1: R3.2, S1.2
- new net VCC: C1.1, J4.2.1, U1.VIN
- net !RESET: now also J2.5; no longer J4.5
- net +5V: now also J2.2; no longer J4.2
- net 0V: now also J2.1, J4.1.1; no longer J4.1
- net PWR_RPI_CNTL: now also J2.9; no longer J4.9
- net RX0: now also J2.7, R7.2, U2A.O; no longer J4.7, U2B.I
- net RX2: now also J2.4; no longer J4.4
- net SHUTDOWN_CNTL: now also J2.10, Q3.D, R4.2; no longer J4.10
- net TX0: now also J2.6, U2B.I; no longer J4.6, R7.2, U2A.O
- net TX2: now also J2.3; no longer J4.3
- net UPDI: now also J2.8; no longer J4.8
Other:
- note added: "7/19/20"
- note added: "SWAP M4809 FOR 128DA28 UART0 CROSSOVER"
- note added: "^1"
- note removed: "SET WEAK PULLUP"
- moved on the sheet: J3, R3

Commit message: PiUpdi: review
Parts:
- added R12: 3.01k, R-C:R0805
- R10: value 3.01k -> 1.82k
- R11: value 1.82k -> 3.01k
- R3: value 1k -> 100k
- R4: value 10k -> 1k
- R7: value 3.01k -> 182
- R8: value 10k -> 3.01k
- R9: value 3.01k -> 10k
- renumbered C7 to C6, U5 to U3
Connections:
- new net N$3: J5.BCM6, R6.2
- net !UPDI_: now also R9.1; no longer R8.1
- net +3V3: now also R10.1; no longer R11.1
- net +5V: now also R11.1, R3.1, R8.1; no longer R4.1, R7.1, R9.1
- net 0V: now also R9.2; no longer R8.2
- net N$1: now also R4.2; no longer R3.2
- net N$2: now also R7.1; no longer R6.1
- net N$4: now also R11.2, R12.2; no longer R10.2, R9.2
- net RX0: now also R8.2; no longer R7.2
- net RX_: now also R10.2; no longer R11.2
- net SHUTDOWN: now also R6.1; no longer J5.BCM6
- net SHUTDOWN_CNTL: now also R3.2, R4.1; no longer R3.1, R4.2
- net UPDI: now also R12.1; no longer R10.1
- net UPDI_: now also R7.2; no longer R6.2
Other:
- moved on the sheet: R10, R11, R3, R4, R6, R7, R8, R9
