File: RPUusb/14145.brd (EAGLE design)
At the start: 71.1 x 33 mm, 50 parts, among them J1 B, J2 40 PIN HDR, Q1 DMB, Q2 K3N, Q3 K3N, U1 CP2105, U2 KB33, U3 ATMEGA328PB-AU, Y1 12MHz

Commit message: RPUusb: pin names on schematic match io_enum
Connections:
- net !CTS0 renamed USB_UART0_!CTS
- net !RTS0 renamed USB_UART0_!RTS
- net !RTS1 renamed USB_UART1_!RTS
- net !SS! renamed !CE00!
- net !SS1! renamed !CE10!
- net 17 renamed BCM44
- net 18 renamed BCM27
- net 2 renamed BCM23
- net 21 renamed BCM22
- net 3 renamed BCM24
- net 8 renamed BCM5
- net 9 renamed BCM26
- net OCOA renamed BCM12_PWM0
- net OCOB renamed BCM13_PWM1
- net RX0 renamed USB_UART0_RX
- net RX1 renamed USB_UART1_RX
- net SCL1 renamed ID_SC
- net SDA1 renamed ID_SD
- net TX0 renamed USB_UART0_TX
- net TX1 renamed USB_UART1_TX
Changed lines of the file:
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@@
 <wire x1="48.514" y1="15.621" x2="48.895" y2="16.002" width="0.3048" layer="1"/>
 </signal>
-<signal name="!SS!">
+<signal name="!CE00!">
 <contactref element="U3" pad="14"/>
 <contactref element="J2" pad="24"/>
@@
 <via x="42.672" y="14.097" extent="1-16" drill="0.4064"/>
 </signal>
-<signal name="TX1">
+<signal name="USB_UART1_TX">
 <contactref element="U3" pad="30"/>
 <contactref element="U1" pad="21"/>
@@
 <wire x1="46.736" y1="12.827" x2="47.117" y2="12.446" width="0.3048" layer="1"/>
 </signal>
-<signal name="SDA1">
+<signal name="ID_SD">
 <contactref element="U3" pad="3"/>
 <contactref element="J2" pad="27"/>
@@
 <wire x1="31.242" y1="5.842" x2="30.48" y2="5.08" width="0.2032" layer="16"/>
 </signal>
-<signal name="SCL1">
+<signal name="ID_SC">
 <contactref element="U3" pad="6"/>
 <contactref element="J2" pad="28"/>
@@
 <wire x1="48.514" y1="18.669" x2="48.641" y2="18.669" width="0.2032" layer="1"/>
 </signal>
-<signal name="RX1">
+<signal name="USB_UART1_RX">
 <contactref element="U3" pad="31"/>
 <contactref element="U1" pad="20"/>
@@
 <wire x1="12.485" y1="16.725" x2="11.557" y2="17.653" width="0.2032" layer="1"/>
 </signal>
-<signal name="!RTS1">
+<signal name="USB_UART1_!RTS">
 <contactref element="U1" pad="19"/>
 <contactref element="C10" pad="1"/>
@@
 <wire x1="19.812" y1="25.654" x2="19.812" y2="27.178" width="0.2032" layer="1"/>
 </signal>
-<signal name="TX0">
+<signal name="USB_UART0_TX">
 <contactref element="U1" pad="13"/>
 <contactref element="J2" pad="8"/>
@@
 <wire x1="20.848" y1="21.229" x2="21.082" y2="21.463" width="0.2032" layer="1"/>
 </signal>
-<signal name="RX0">
+<signal name="USB_UART0_RX">
 <contactref element="U1" pad="12"/>
 <contactref element="J2" pad="10"/>
@@
 <wire x1="26.162" y1="22.352" x2="24.511" y2="20.701" width="0.2032" layer="16"/>
 </signal>
-<signal name="!RTS0">
+<signal name="USB_UART0_!RTS">
 <contactref element="U1" pad="11"/>
 <contactref element="J2" pad="11"/>
@@
 <wire x1="51.308" y1="5.588" x2="50.8" y2="5.08" width="0.2032" layer="16"/>
 </signal>
-<signal name="!CTS0">
+<signal name="USB_UART0_!CTS">
 <contactref element="U1" pad="10"/>
 <contactref element="J2" pad="36"/>
@@
 <wire x1="17.784" y1="18.499" x2="18.542" y2="17.741" width="0.2032" layer="1"/>
 </signal>
-<signal name="OCOA">
+<signal name="BCM12_PWM0">
 <contactref element="U3" pad="10"/>
 <contactref element="J2" pad="32"/>
@@
 <wire x1="25.4" y1="3.556" x2="25.4" y2="2.54" width="0.2032" layer="16"/>
 </signal>
-<signal name="OCOB">
+<signal name="BCM13_PWM1">
 <contactref element="J2" pad="33"/>
 <contactref element="U3" pad="9"/>
@@
 <wire x1="16.002" y1="2.54" x2="15.24" y2="2.54" width="0.2032" layer="1"/>
 </signal>
-<signal name="!SS1!">
+<signal name="!CE10!">
 <contactref element="U3" pad="19"/>
 <contactref element="J2" pad="12"/>
@@
 <wire x1="17.78" y1="3.683" x2="17.78" y2="2.54" width="0.2032" layer="16"/>
 </signal>
-<signal name="2">
+<signal name="BCM23">
 <contactref element="U3" pad="25"/>
 <contactref element="J2" pad="16"/>
@@
 <wire x1="45.72" y1="3.048" x2="45.72" y2="2.54" width="0.2032" layer="1"/>
 </signal>
-<signal name="3">
+<signal name="BCM24">
 <contactref element="U3" pad="26"/>
 <contactref element="J2" pad="18"/>
@@
 <wire x1="43.561" y1="2.54" x2="43.18" y2="2.54" width="0.2032" layer="16"/>
 </signal>
-<signal name="17">
+<signal name="BCM44">
 <contactref element="U3" pad="1"/>
 <contactref element="J2" pad="7"/>
@@
 <wire x1="60.68065" y1="19.05" x2="61.722" y2="19.05" width="0.2032" layer="1"/>
 </signal>
-<signal name="18">
+<signal name="BCM27">
 <contactref element="U3" pad="2"/>
 <contactref element="J2" pad="13"/>
@@
 <wire x1="49.403" y1="6.223" x2="48.26" y2="5.08" width="0.2032" layer="1"/>
 </signal>
-<signal name="21">
+<signal name="BCM22">
 <contactref element="U3" pad="11"/>
 <contactref element="J2" pad="15"/>
@@
 <wire x1="46.609" y1="20.447" x2="46.355" y2="20.701" width="0.2032" layer="16"/>
 </signal>
-<signal name="8">
+<signal name="BCM5">
 <contactref element="U3" pad="12"/>
 <contactref element="J2" pad="29"/>
@@
 <wire x1="27.94" y1="16.002" x2="27.94" y2="5.08" width="0.2032" layer="16"/>
 </signal>
-<signal name="9">
+<signal name="BCM26">
 <contactref element="U3" pad="13"/>
 <contactref element="J2" pad="37"/>
