File: RPUusb/14145.sch (EAGLE design)
At the start: 50 parts, among them J1 B, J2 40 PIN HDR, Q1 DMB, Q2 K3N, Q3 K3N, U1 CP2105, U2 KB33, U3 ATMEGA328PB-AU, Y1 12MHz

Commit message: RPUusb: pin names on schematic match io_enum
Connections:
- net !CTS0 renamed USB_UART0_!CTS
- net !RTS0 renamed USB_UART0_!RTS
- net !RTS1 renamed USB_UART1_!RTS
- net !SS! renamed !CE00!
- net !SS1! renamed !CE10!
- net 17 renamed BCM44
- net 18 renamed BCM27
- net 2 renamed BCM23
- net 21 renamed BCM22
- net 3 renamed BCM24
- net 8 renamed BCM5
- net 9 renamed BCM26
- net OCOA renamed BCM12_PWM0
- net OCOB renamed BCM13_PWM1
- net RX0 renamed USB_UART0_RX
- net RX1 renamed USB_UART1_RX
- net SCL1 renamed ID_SC
- net SDA1 renamed ID_SD
- net TX0 renamed USB_UART0_TX
- net TX1 renamed USB_UART1_TX
Other:
- note added: "NOTE: RX & TX CROSS OVER AT TRANSCEIVER"
- note removed: "0"
- note removed: "1"
- note removed: "10"
- note removed: "11"
- note removed: "12"
- note removed: "13"
- note removed: "14"
- note removed: "15"
- note removed: "16"
- note removed: "17"
- note removed: "18"
- note removed: "19"
- note removed: "2"
- note removed: "20"
- note removed: "21"
- note removed: "22"
- note removed: "23"
- note removed: "3"
- note removed: "4"
- note removed: "5"
- note removed: "6"
- note removed: "7"
- note removed: "8"
- note removed: "9"
Changed lines of the file:
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@@
 328, FULL BUS CONT</text>
 <text x="320.548" y="16.51" size="1.778" layer="98">11/22/15</text>
-<wire x1="121.412" y1="182.88" x2="129.286" y2="182.88" width="0.4064" layer="98"/>
-<wire x1="129.286" y1="182.88" x2="128.27" y2="182.118" width="0.4064" layer="98"/>
-<wire x1="129.286" y1="182.88" x2="128.27" y2="183.642" width="0.4064" layer="98"/>
-<wire x1="121.412" y1="205.74" x2="129.286" y2="205.74" width="0.4064" layer="98"/>
-<wire x1="129.286" y1="205.74" x2="128.27" y2="204.978" width="0.4064" layer="98"/>
-<wire x1="129.286" y1="205.74" x2="128.27" y2="206.502" width="0.4064" layer="98"/>
-<wire x1="129.032" y1="203.2" x2="121.158" y2="203.2" width="0.4064" layer="98"/>
-<wire x1="121.158" y1="203.2" x2="122.174" y2="203.962" width="0.4064" layer="98"/>
-<wire x1="121.158" y1="203.2" x2="122.174" y2="202.438" width="0.4064" layer="98"/>
+<wire x1="129.032" y1="182.88" x2="136.906" y2="182.88" width="0.4064" layer="98"/>
+<wire x1="136.906" y1="182.88" x2="135.89" y2="182.118" width="0.4064" layer="98"/>
+<wire x1="136.906" y1="182.88" x2="135.89" y2="183.642" width="0.4064" layer="98"/>
+<wire x1="131.572" y1="205.74" x2="139.446" y2="205.74" width="0.4064" layer="98"/>
+<wire x1="139.446" y1="205.74" x2="138.43" y2="204.978" width="0.4064" layer="98"/>
+<wire x1="139.446" y1="205.74" x2="138.43" y2="206.502" width="0.4064" layer="98"/>
+<wire x1="139.192" y1="203.2" x2="131.318" y2="203.2" width="0.4064" layer="98"/>
+<wire x1="131.318" y1="203.2" x2="132.334" y2="203.962" width="0.4064" layer="98"/>
+<wire x1="131.318" y1="203.2" x2="132.334" y2="202.438" width="0.4064" layer="98"/>
 <text x="23.622" y="18.796" size="1.778" layer="98">CRYSTAL:
 ECS-120-20-3X-TR
@@
 <text x="290.068" y="25.908" size="1.6764" layer="98">ICP1 TO TP</text>
 <text x="320.548" y="26.67" size="1.778" layer="98">1/14/17</text>
-<wire x1="129.032" y1="180.34" x2="121.158" y2="180.34" width="0.4064" layer="98"/>
-<wire x1="121.158" y1="180.34" x2="122.174" y2="181.102" width="0.4064" layer="98"/>
-<wire x1="121.158" y1="180.34" x2="122.174" y2="179.578" width="0.4064" layer="98"/>
+<wire x1="136.652" y1="180.34" x2="128.778" y2="180.34" width="0.4064" layer="98"/>
+<wire x1="128.778" y1="180.34" x2="129.794" y2="181.102" width="0.4064" layer="98"/>
+<wire x1="128.778" y1="180.34" x2="129.794" y2="179.578" width="0.4064" layer="98"/>
 <text x="320.548" y="31.75" size="1.778" layer="98">8/26/19</text>
 <text x="290.068" y="30.988" size="1.6764" layer="98">SILAB USB, MCU IS FOR
 DBUG ON 40 PIN R-PI HDR</text>
 <text x="282.702" y="32.004" size="2.54" layer="98">^5</text>
-<text x="110.744" y="108.458" size="1.778" layer="98">0</text>
-<text x="110.744" y="105.918" size="1.778" layer="98">1</text>
-<text x="110.744" y="103.378" size="1.778" layer="98">2</text>
-<text x="110.744" y="100.838" size="1.778" layer="98">3</text>
-<text x="143.764" y="98.298" size="1.778" layer="98">4</text>
-<text x="143.764" y="95.758" size="1.778" layer="98">5</text>
-<text x="110.744" y="93.218" size="1.778" layer="98">6</text>
-<text x="110.744" y="90.678" size="1.778" layer="98">7</text>
-<text x="113.284" y="62.738" size="1.778" layer="98">8</text>
-<text x="113.284" y="60.198" size="1.778" layer="98">9</text>
-<text x="113.284" y="57.658" size="1.778" layer="98">10</text>
-<text x="128.524" y="55.118" size="1.778" layer="98">11</text>
-<text x="128.524" y="52.578" size="1.778" layer="98">12</text>
-<text x="128.524" y="50.038" size="1.778" layer="98">13</text>
-<text x="115.824" y="83.058" size="1.778" layer="98">14</text>
-<text x="115.824" y="85.598" size="1.778" layer="98">15</text>
-<text x="115.824" y="80.518" size="1.778" layer="98">16</text>
-<text x="115.824" y="77.978" size="1.778" layer="98">17</text>
-<text x="115.824" y="75.438" size="1.778" layer="98">18</text>
-<text x="115.824" y="72.898" size="1.778" layer="98">19</text>
-<text x="115.824" y="70.358" size="1.778" layer="98">20</text>
-<text x="115.824" y="67.818" size="1.778" layer="98">21</text>
-<text x="44.704" y="47.498" size="1.778" layer="98">22</text>
-<text x="44.704" y="44.958" size="1.778" layer="98">23</text>
 <text x="261.62" y="221.742" size="2.54" layer="98">SBC (R-PI) HDR FOR DEBUGING RPU TARGET</text>
 <text x="84.582" y="158.496" size="1.778" layer="98">Silicon Labs factory default
 VID: 0x10C4
 PID: 0xEA7A</text>
-<wire x1="250.952" y1="198.12" x2="258.826" y2="198.12" width="0.4064" layer="98"/>
-<wire x1="258.826" y1="198.12" x2="257.81" y2="197.358" width="0.4064" layer="98"/>
-<wire x1="258.826" y1="198.12" x2="257.81" y2="198.882" width="0.4064" layer="98"/>
-<wire x1="335.788" y1="167.64" x2="343.662" y2="167.64" width="0.4064" layer="98"/>
-<wire x1="343.662" y1="167.64" x2="342.646" y2="166.878" width="0.4064" layer="98"/>
-<wire x1="343.662" y1="167.64" x2="342.646" y2="168.402" width="0.4064" layer="98"/>
+<wire x1="240.792" y1="198.12" x2="248.666" y2="198.12" width="0.4064" layer="98"/>
+<wire x1="248.666" y1="198.12" x2="247.65" y2="197.358" width="0.4064" layer="98"/>
+<wire x1="248.666" y1="198.12" x2="247.65" y2="198.882" width="0.4064" layer="98"/>
+<wire x1="345.948" y1="167.64" x2="353.822" y2="167.64" width="0.4064" layer="98"/>
+<wire x1="353.822" y1="167.64" x2="352.806" y2="166.878" width="0.4064" layer="98"/>
+<wire x1="353.822" y1="167.64" x2="352.806" y2="168.402" width="0.4064" layer="98"/>
+<text x="346.202" y="199.136" size="1.778" layer="98">NOTE: RX &amp; TX CROSS
+OVER AT TRANSCEIVER</text>
 </plain>
 <instances>
@@
 </segment>
 </net>
-<net name="!SS!" class="0">
+<net name="!CE00!" class="0">
 <segment>
 <pinref part="U3" gate="G$1" pin="(!SS!/OC1B)PB2"/>
@@
 </segment>
 </net>
-<net name="TX1" class="0">
-<segment>
-<label x="106.68" y="83.82" size="1.27" layer="91" xref="yes"/>
+<net name="USB_UART1_TX" class="0">
+<segment>
+<label x="104.14" y="86.36" size="1.27" layer="91" xref="yes"/>
 <pinref part="U3" gate="G$1" pin="(RXD)PD0"/>
-<wire x1="99.06" y1="86.36" x2="101.6" y2="86.36" width="0.1524" layer="91"/>
-<wire x1="101.6" y1="86.36" x2="104.14" y2="83.82" width="0.1524" layer="91"/>
-<wire x1="104.14" y1="83.82" x2="106.68" y2="83.82" width="0.1524" layer="91"/>
+<wire x1="99.06" y1="86.36" x2="104.14" y2="86.36" width="0.1524" layer="91"/>
 </segment>
 <segment>
@@
 </segment>
 </net>
-<net name="SDA1" class="0">
+<net name="ID_SD" class="0">
 <segment>
 <pinref part="U3" gate="G$1" pin="PE0(SDA1/ICP4)"/>
@@
 </segment>
 </net>
-<net name="SCL1" class="0">
+<net name="ID_SC" class="0">
 <segment>
 <pinref part="U3" gate="G$1" pin="PE1(SCL1/T4)"/>
@@
 </segment>
 </net>
-<net name="RX1" class="0">
-<segment>
-<label x="106.68" y="86.36" size="1.27" layer="91" xref="yes"/>
+<net name="USB_UART1_RX" class="0">
+<segment>
+<label x="104.14" y="83.82" size="1.27" layer="91" xref="yes"/>
 <pinref part="U3" gate="G$1" pin="(TXD)PD1"/>
-<wire x1="99.06" y1="83.82" x2="101.6" y2="83.82" width="0.1524" layer="91"/>
-<wire x1="101.6" y1="83.82" x2="104.14" y2="86.36" width="0.1524" layer="91"/>
-<wire x1="104.14" y1="86.36" x2="106.68" y2="86.36" width="0.1524" layer="91"/>
+<wire x1="99.06" y1="83.82" x2="104.14" y2="83.82" width="0.1524" layer="91"/>
 </segment>
 <segment>
@@
 </segment>
 </net>
-<net name="!RTS1" class="0">
+<net name="USB_UART1_!RTS" class="0">
 <segment>
 <pinref part="U1" gate="G$1" pin="!RTS!_SCI"/>
@@
 </segment>
 </net>
-<net name="TX0" class="0">
+<net name="USB_UART0_TX" class="0">
 <segment>
 <pinref part="U1" gate="G$1" pin="TX_ECI"/>
@@
 </segment>
 </net>
-<net name="RX0" class="0">
+<net name="USB_UART0_RX" class="0">
 <segment>
 <pinref part="U1" gate="G$1" pin="RX_ECI"/>
@@
 </segment>
 </net>
-<net name="!RTS0" class="0">
+<net name="USB_UART0_!RTS" class="0">
 <segment>
 <pinref part="U1" gate="G$1" pin="!RTS!_ECI"/>
@@
 </segment>
 </net>
-<net name="!CTS0" class="0">
+<net name="USB_UART0_!CTS" class="0">
 <segment>
 <pinref part="U1" gate="G$1" pin="!CTS!_ECI"/>
@@
 </segment>
 </net>
-<net name="OCOA" class="0">
+<net name="BCM12_PWM0" class="0">
 <segment>
 <pinref part="U3" gate="G$1" pin="(OC0A)PD6"/>
@@
 </segment>
 </net>
-<net name="OCOB" class="0">
+<net name="BCM13_PWM1" class="0">
 <segment>
 <pinref part="J2" gate="G$1" pin="BCM13/PWM1"/>
@@
 </segment>
 </net>
-<net name="!SS1!" class="0">
+<net name="!CE10!" class="0">
 <segment>
 <pinref part="U3" gate="G$1" pin="(ICP3/!SS1!)PE2"/>
@@
 </segment>
 </net>
-<net name="2" class="0">
+<net name="BCM23" class="0">
 <segment>
 <pinref part="U3" gate="G$1" pin="(A2)PC2"/>
@@
 </segment>
 </net>
-<net name="3" class="0">
+<net name="BCM24" class="0">
 <segment>
 <pinref part="U3" gate="G$1" pin="(A3)PC3"/>
@@
 </segment>
 </net>
-<net name="17" class="0">
+<net name="BCM44" class="0">
 <segment>
 <pinref part="U3" gate="G$1" pin="(INT1/OC2B)PD3"/>
@@
 </segment>
 </net>
-<net name="18" class="0">
+<net name="BCM27" class="0">
 <segment>
 <pinref part="U3" gate="G$1" pin="(T0)PD4"/>
@@
 </segment>
 </net>
-<net name="21" class="0">
+<net name="BCM22" class="0">
 <segment>
 <pinref part="U3" gate="G$1" pin="PD7"/>
@@
 </segment>
 </net>
-<net name="8" class="0">
+<net name="BCM5" class="0">
 <segment>
 <pinref part="U3" gate="G$1" pin="(ICP1)PB0"/>
@@
 </segment>
 </net>
-<net name="9" class="0">
+<net name="BCM26" class="0">
 <segment>
 <pinref part="U3" gate="G$1" pin="(OC1A)PB1"/>
