File: Buck/20226.sch (EAGLE design)
At the start: 14 parts, among them U2 AP64352Q

Commit message: Buck: looking at the inductor
Other:
- note added: "SRP7028A is 2626 size, it fits on SRP7030 size 2831"
Changed lines of the file:
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@@
 <text x="120.396" y="101.092" size="1.778" layer="98">freq [kHz] = 100000 / (100[kOhm])   = 1MegHz</text>
 <text x="112.776" y="141.732" size="2.54" layer="98">7V to 40V</text>
+<text x="120.396" y="96.012" size="1.778" layer="98">SRP7028A is 2626 size, it fits on SRP7030 size 2831</text>
 </plain>
 <instances>
